File: KiCad/Humanoide/Humanoide.sch (KiCad schematic (older format))
At the start: 115 parts, among them CON1 SPI, IC1 CP2102, P1 CONN_01X03, P10 USB_OTG, P11 SRV9, P12 SRV10, P13 SRV11, P14 SRV12, P15 SRV13, P16 SRV14, P17 SRV15, P18 SRV16, P19 SRV17, P2 SRV1, P20 SRV18, P21 SRV19, P22 SRV20, P23 I2C, P24 UART, P25 V_BATT, P26 USB_BT, P3 SRV2, P4 SRV3, P5 SRV4, P6 SRV5, P7 SRV6, P8 SRV7, P9 SRV8, Q1 IRF7842PBF, SW1 SW_PUSH, U1 LM3940IMP, U2 ATSAM3X8EA-AU, X1 CSTCE 12MHz, Y1 32.768kHz

Commit message: Kicad 3D model changed
Parts:
- P26: footprint Humanoide_lib:USB-B -> Humanoide_lib:USB-A-SMD
Changed lines of the file:
@@
 F 0 "P26" H 8050 6100 50  0000 C CNN
 F 1 "USB_BT" H 7800 6500 50  0000 C CNN
-F 2 "Humanoide_lib:USB-B" V 7800 6200 50  0001 C CNN
+F 2 "Humanoide_lib:USB-A-SMD" V 7800 6200 50  0001 C CNN
 F 3 "" V 7800 6200 50  0000 C CNN
 	1    7850 6300

Commit message: Schematic added
Parts:
- D10, D2, D6, D7, D8, D9: symbol LED -> LED-RESCUE-Humanoide
- P10: symbol USB_OTG -> USB_OTG-RESCUE-Humanoide
- P26: symbol USB_B -> USB_B-RESCUE-Humanoide
Changed lines of the file:
@@
 EESchema Schematic File Version 2
+LIBS:Humanoide-rescue
 LIBS:power
 LIBS:device
@@
 $EndComp
 $Comp
-L LED D2
+L LED-RESCUE-Humanoide D2
 U 1 1 578003D2
 P 4300 1700
@@
 RX1
 $Comp
-L LED D6
+L LED-RESCUE-Humanoide D6
 U 1 1 57843CAB
 P 9700 9850
@@
 $EndComp
 $Comp
-L LED D7
+L LED-RESCUE-Humanoide D7
 U 1 1 57843D3F
 P 10000 9850
@@
 $EndComp
 $Comp
-L LED D8
+L LED-RESCUE-Humanoide D8
 U 1 1 57843E0B
 P 10300 9850
@@
 $EndComp
 $Comp
-L USB_OTG P10
+L USB_OTG-RESCUE-Humanoide P10
 U 1 1 578D79B5
 P 1500 4400
@@
 NoConn ~ 10300 5450
 $Comp
-L LED D9
+L LED-RESCUE-Humanoide D9
 U 1 1 57C4E7AB
 P 10800 9900
@@
 $EndComp
 $Comp
-L LED D10
+L LED-RESCUE-Humanoide D10
 U 1 1 57C4E7B7
 P 11100 9900
@@
 	3350 4800 3350 4900
 $Comp
-L USB_B P26
+L USB_B-RESCUE-Humanoide P26
 U 1 1 57BB9DA8
 P 7850 6300
